File: kicad/BatteryChecker.kicad_sch (KiCad schematic)
At the start: 19 parts, among them M5Stick_C_Plus? M5Stick_C_Plus, Q1 TC004B, Q2 2SC1815

Commit message: * MCP4725/4726の品番を追加 * I2Cアドレスを明記 * MCP4725のA0接続先の接続漏れを修正 * AE-ADS1015に関する補足を追加
Parts:
- U?: value MCP4725 -> AE-MCP4725(MCP4725A0T-E/CH)
- U?: value ADS1015IDGS -> AE-ADS1015(akizuki)
- U?: value MCP4726 -> AE-MCP4726(MCP4726A0T-E/CH)
Connections:
- net +5V: now also U?.6 (A0)
Other:
- note added: "ADDRが変換基板で10kΩプルダウン済"
- note added: "VDD接続でアドレス61h"
- note added: "アドレス60h固定"
Changed lines of the file:
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@@
   (junction (at 215.9 43.18) (diameter 0) (color 0 0 0 0)
   )
+  (junction (at 82.55 81.28) (diameter 0) (color 0 0 0 0)
+  )
   (junction (at 53.34 48.26) (diameter 0) (color 0 0 0 0)
   )
@@
     (stroke (width 0) (type default) (color 0 0 0 0))
   )
+  (wire (pts (xy 72.39 91.44) (xy 69.85 91.44))
+    (stroke (width 0) (type default) (color 0 0 0 0))
+  )
   (wire (pts (xy 95.25 88.9) (xy 92.71 88.9))
     (stroke (width 0) (type default) (color 0 0 0 0))
@@
     (stroke (width 0) (type default) (color 0 0 0 0))
   )
+  (wire (pts (xy 69.85 91.44) (xy 69.85 81.28))
+    (stroke (width 0) (type default) (color 0 0 0 0))
+  )
   (wire (pts (xy 172.72 127) (xy 177.8 127))
     (stroke (width 0) (type default) (color 0 0 0 0))
@@
     (stroke (width 0) (type default) (color 0 0 0 0))
   )
+  (wire (pts (xy 69.85 81.28) (xy 82.55 81.28))
+    (stroke (width 0) (type default) (color 0 0 0 0))
+  )
   (wire (pts (xy 64.77 39.37) (xy 72.39 39.37))
     (stroke (width 0) (type default) (color 0 0 0 0))
@@
   (wire (pts (xy 187.96 63.5) (xy 187.96 72.39))
     (stroke (width 0) (type default) (color 0 0 0 0))
+  )
+  (text "ADDRが変換基板で10kΩプルダウン済" (at 129.54 55.88 0)
+    (effects (font (size 1.27 1.27)) (justify left bottom))
+  )
+  (text "VDD接続でアドレス61h" (at 57.15 97.79 0)
+    (effects (font (size 1.27 1.27)) (justify left bottom))
+  )
+  (text "アドレス60h固定" (at 91.44 35.56 0)
+    (effects (font (size 1.27 1.27)) (justify left bottom))
   )
   (symbol (lib_name "+5V_2") (lib_id "power:+5V") (at 82.55 27.94 0) (unit 1)
@@
       (effects (font (size 1.27 1.27)) hide)
     )
-    (property "Value" "MCP4725" (id 1) (at 95.25 81.28 0))
+    (property "Value" "AE-MCP4725(MCP4725A0T-E/CH)" (id 1) (at 100.33 81.28 0))
     (property "Footprint" "Package_TO_SOT_SMD:SOT-23-6" (id 2) (at 82.55 95.25 0)
       (effects (font (size 1.27 1.27)) hide)
@@
       (effects (font (size 1.27 1.27)) (justify left) hide)
     )
-    (property "Value" "ADS1015IDGS" (id 1) (at 127.7494 31.75 0)
+    (property "Value" "AE-ADS1015(akizuki)" (id 1) (at 127.7494 31.75 0)
       (effects (font (size 1.27 1.27)) (justify left))
     )
@@
       (effects (font (size 1.27 1.27)) hide)
     )
-    (property "Value" "MCP4726" (id 1) (at 95.25 31.75 0))
+    (property "Value" "AE-MCP4726(MCP4726A0T-E/CH)" (id 1) (at 100.33 31.75 0))
     (property "Footprint" "Package_TO_SOT_SMD:SOT-23-6" (id 2) (at 82.55 45.72 0)
       (effects (font (size 1.27 1.27)) hide)
@@
     (pin "6")
   )
+  (symbol (lib_id "Graphic:SYM_Arrow45_Small") (at 138.43 52.07 180) (unit 1)
+    (in_bom yes) (on_board yes) (fields_autoplaced)
+    (property "Reference" "#SYM?" (id 0) (at 134.112 53.086 0)
+      (effects (font (size 1.27 1.27)) hide)
+    )
+    (property "Value" "SYM_Arrow45_Small" (id 1) (at 138.43 49.784 0)
+      (effects (font (size 1.27 1.27)) hide)
+    )
+    (property "Footprint" "" (id 2) (at 138.43 52.07 0)
+      (effects (font (size 1.27 1.27)) hide)
+    )
+    (property "Datasheet" "~" (id 3) (at 138.43 52.07 0)
+      (effects (font (size 1.27 1.27)) hide)
+    )
+  )
   (symbol (lib_id "power:GND") (at 251.46 149.86 0) (unit 1)
     (in_bom yes) (on_board yes) (fields_autoplaced)
@@
     (pin "1")
     (pin "2")
+  )
+  (symbol (lib_id "Graphic:SYM_Arrow45_Small") (at 71.12 93.98 90) (unit 1)
+    (in_bom yes) (on_board yes) (fields_autoplaced)
+    (property "Reference" "#SYM?" (id 0) (at 70.104 89.662 0)
+      (effects (font (size 1.27 1.27)) hide)
+    )
+    (property "Value" "SYM_Arrow45_Small" (id 1) (at 73.406 93.98 0)
+      (effects (font (size 1.27 1.27)) hide)
+    )
+    (property "Footprint" "" (id 2) (at 71.12 93.98 0)
+      (effects (font (size 1.27 1.27)) hide)
+    )
+    (property "Datasheet" "~" (id 3) (at 71.12 93.98 0)
+      (effects (font (size 1.27 1.27)) hide)
+    )
   )
   (symbol (lib_name "GND_3") (lib_id "power:GND") (at 82.55 50.8 0) (unit 1)
@@
       (reference "#SYM?") (unit 1) (value "V3") (footprint "")
     )
+    (path "/d79a6777-5713-496d-9f38-50f4810229ef"
+      (reference "#SYM?") (unit 1) (value "SYM_Arrow45_Small") (footprint "")
+    )
+    (path "/e7db7406-add8-4e6b-840c-533a0179faa1"
+      (reference "#SYM?") (unit 1) (value "SYM_Arrow45_Small") (footprint "")
+    )
     (path "/ec2afb69-73ad-4372-b948-7791f355e7f0"
       (reference "#SYM?") (unit 1) (value "V1") (footprint "")
@@
     )
     (path "/4189f762-e0f9-4d46-a0d6-c61e4b31bf4c"
-      (reference "U?") (unit 1) (value "MCP4725") (footprint "Package_TO_SOT_SMD:SOT-23-6")
+      (reference "U?") (unit 1) (value "AE-MCP4725(MCP4725A0T-E/CH)") (footprint "Package_TO_SOT_SMD:SOT-23-6")
     )
     (path "/adf702a1-9eac-4d38-9c51-2a391d3bf372"
-      (reference "U?") (unit 1) (value "ADS1015IDGS") (footprint "Package_SO:TSSOP-10_3x3mm_P0.5mm")
+      (reference "U?") (unit 1) (value "AE-ADS1015(akizuki)") (footprint "Package_SO:TSSOP-10_3x3mm_P0.5mm")
     )
     (path "/c88f2570-9379-4b76-8208-061e50d68e9b"
-      (reference "U?") (unit 1) (value "MCP4726") (footprint "Package_TO_SOT_SMD:SOT-23-6")
-    )
-  )
+      (reference "U?") (unit 1) (value "AE-MCP4726(MCP4726A0T-E/CH)") (footprint "Package_TO_SOT_SMD:SOT-23-6")
+    )
+  )
